File: PCB/keyboard-pcb.kicad_pcb (KiCad board)
At the start: 2 copper layers, 381 x 131 mm, 181 parts, among them J1 Conn_01x05_Pin, U1 Raspberry_Pi_Pico

Commit message: Modified JOURNAL.md
Parts:
- gave numbers to parts that had none: 1
- renumbered ESC to MX1, F9 to MX10, F10 to MX11, F11 to MX12, F12 to MX13, PRTSC to MX14, SCRLK to MX15, PAUSE to MX16, ` to MX17, 1 to MX18, 2 to MX19, F1 to MX2, 3 to MX20, 4 to MX21, 5 to MX22, 6 to MX23, 7 to MX24, 8 to MX25, 9 to MX26, 0 to MX27, - to MX28, + to MX29, F2 to MX3, BKSPC to MX30, INSERT to MX31, HOME to MX32, PGUP to MX33, TAB to MX34, Q to MX35, W to MX36, E to MX37, R to MX38, T to MX39, F3 to MX4, Y to MX40, U to MX41, I to MX42, O to MX43, P to MX44, { to MX45, } to MX46, | to MX47, DEL to MX48, END to MX49, F4 to MX5, PGDN to MX50, CAPS to MX51, A to MX52, S to MX53, D to MX54, F to MX55, G to MX56, H to MX57, J to MX58, K to MX59, F5 to MX6, L to MX60, : to MX61, " to MX62, ENTER to MX63, L_SHFT to MX64, Z to MX65, X to MX66, C to MX67, V to MX68, B to MX69, F6 to MX7, N to MX70, M to MX71, < to MX72, > to MX73, R_SHFT to MX75, UP to MX76, L_CTRL to MX78, WIN to MX79, F7 to MX8, ALT to MX80, SPACE to MX81, ALT to MX82, FN to MX83, MENU to MX84, R_CTRL to MX85, RIGHT to MX86, DOWN to MX87, LEFT to MX88, F8 to MX9
Connections:
- U1 pad 23: Row 2 -> unconnected-(U1-GND-Pad23)
- U1 pad 24: Row 3 -> Row 2
- U1 pad 25: unconnected-(U1-GPIO19-Pad25) -> Row 3
Routing:
- net Row 3: track 369.6 -> 381.1 mm, vias 0 -> 2
- net Row 2: track 366.8 -> 372.0 mm, vias 0 -> 1

Commit message: Modified whole case, added accents (jinx from arcane reference), connected all gnd pins
Parts:
- added REF**: MountingHole_2.2mm_M2, MountingHole:MountingHole_2.2mm_M2, F.Cu at (392.9, 154.8)
- added REF**: MountingHole_2.2mm_M2, MountingHole:MountingHole_2.2mm_M2, F.Cu at (140.5, 38.1)
- added REF**: MountingHole_2.2mm_M2, MountingHole:MountingHole_2.2mm_M2, F.Cu at (119.1, 147.6)
- added REF**: MountingHole_2.2mm_M2, MountingHole:MountingHole_2.2mm_M2, F.Cu at (45.2, 35.7)
- added REF**: MountingHole_2.2mm_M2, MountingHole:MountingHole_2.2mm_M2, F.Cu at (316.7, 119.1)
Connections:
- U1 pad 13: unconnected-(U1-GND-Pad13) -> GND
- U1 pad 18: unconnected-(U1-GND-Pad18) -> GND
- U1 pad 23: unconnected-(U1-GND-Pad23) -> GND
- U1 pad 28: unconnected-(U1-GND-Pad28) -> GND
- U1 pad 38: unconnected-(U1-GND-Pad38) -> GND
- U1 pad 42: unconnected-(U1-GND-Pad42) -> GND
- U1 pad 8: unconnected-(U1-GND-Pad8) -> GND
Routing:
- net GND: track 61.4 -> 177.4 mm, vias 0 -> 5
- net Column 2: track 447.8 -> 460.0 mm

Commit message: fixed stuff ig
Parts:
- moved D87 39.1 mm to (364.3, 157.2)
- moved MX86 38.1 mm to (321.5, 147.6)
- moved MX88 38.1 mm to (359.6, 147.6)
- moved D85 37.1 mm to (326.2, 157.2)
- moved U1 2.45 mm to (383.6, 57.1)
Connections:
- U1 pad 34: unconnected-(U1-GPIO28_ADC2-Pad34) -> Column 16
Routing:
- net Column 4: track 950.2 -> 514.9 mm
- net Column 3: track 666.7 -> 474.7 mm
- net Column 7: track 373.8 -> 487.4 mm, vias 4 -> 0
- net Column 8: track 378.5 -> 464.0 mm, vias 1 -> 2
- net Column 9: track 354.9 -> 439.1 mm, vias 3 -> 1
- net Column 13: track 164.5 -> 241.0 mm
- net Column 6: track 421.8 -> 485.8 mm, vias 6 -> 0
- net GND: track 177.4 -> 122.8 mm, vias 5 -> 0
- net Column 10: track 427.4 -> 373.5 mm, vias 2 -> 0
- net Row 0: track 431.4 -> 378.2 mm, vias 0 -> 1
- net SW: track 109.4 -> 56.9 mm, vias 2 -> 1
- net S1B: track 88.4 -> 46.8 mm, vias 2 -> 1
- net Column 5: track 446.1 -> 487.0 mm, vias 10 -> 0
- net 3V3: track 86.4 -> 127.3 mm
- net Column 14: track 141.1 -> 181.9 mm
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